File: tsubaki_lite.kicad_sch (KiCad schematic)
At the start: 48 parts, among them J1 USB_C_Receptacle_USB2.0_16P, J2 Conn_01x02, J3 Conn_01x04, Q1 AO3400A, Q2 AO3400A, Q3 AO3400A, Q4 AO3400A, SW1 SW_SPST, SW2 SW_SPST, SW3 EC12E1240406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

Commit message: rev3
Parts:
- removed U1: CH32X033F8P6, Package_SO:TSSOP-20_4.4x6.5mm_P0.65mm, symbol local:CH32X033F8P6
- added U1: CH32X035F7P6, Package_SO:TSSOP-20_4.4x6.5mm_P0.65mm, symbol local:CH32X035F7P6
- C1, C2, C3: footprint Capacitor_SMD:C_0402_1005Metric -> Capacitor_SMD:C_0805_2012Metric
- L_1_1, L_1_2, L_1_3: footprint LED_SMD:LED_0805_2012Metric_Pad1.15x1.40mm_HandSolder -> LED_SMD:LED_0805_2012Metric
- R1, R10, R12, R14, R15, R16, R2, R3, R4, R5, R7, R8: footprint Resistor_SMD:R_0402_1005Metric -> Resistor_SMD:R_0805_2012Metric
Connections:
- net COL1: now also U1.3 (PC15)
- net COL2: now also U1.2 (PC14)
- net COL3: now also U1.1 (PB12)
- net DCK: now also U1.20 (PC19)
- net DIO: now also U1.19 (PC18)
- net DM: now also U1.17 (PC16)
- net DP: now also U1.18 (PC17)
- net GND: now also U1.15 (GND)
- net LED_CTRL: now also U1.11 (PA5)
- net RESET: now also U1.4 (PC3)
- net ROT_DOWN: now also U1.13 (PA7)
- net ROT_UP: now also U1.14 (PB1)
- net ROW1: now also U1.6 (PA0)
- net RX: now also U1.5 (PC1)
- net TX: now also U1.8 (PA2)
- net VDD: now also U1.16 (VDD)
Other:
- note added: "WCH Link interface SWD (SDI) enabled by default; must be disabled after reset."
- note removed: "WCH Link interface (CH32X033 is only compatible with WCH-LinkE or WCH-LinkW) SWD (SDI) enabled by default; must be disabled after reset."

Commit message: rev4
Parts:
- removed D1: LED, LED_SMD:LED_1206_3216Metric, symbol Device:LED
- removed Q1, Q2, Q3, Q4: AO3400A, Package_TO_SOT_SMD:SOT-23, symbol Transistor_FET:AO3400A
- removed R10, R12, R14, R15, R4, R7, R8: 10K, Resistor_SMD:R_0805_2012Metric, symbol Device:R
- removed R11, R13, R6, R9: 220R, Resistor_SMD:R_0402_1005Metric, symbol Device:R
- added D_1_4, D_1_5, D_1_6: 1N4148, Diode_SMD:D_SOD-123, symbol Device:D
- added L_1_4: LED_Small, LED_SMD:LED_0805_2012Metric, symbol Device:LED_Small
- added R_1_4: 560R, Resistor_SMD:R_0402_1005Metric, symbol Device:R
- added SW_1_4: MX-compatible, Button_Switch_Keyboard:SW_Cherry_MX_1.00u_PCB, symbol Switch:SW_Push
- added U2: USBLC6-2SC6, Package_TO_SOT_SMD:SOT-23-6, symbol Power_Protection:USBLC6-2SC6
- renumbered D2 to D1
Connections:
- net COL1: now also U1.1 (PB12); no longer U1.3 (PC15)
- net COL3: now also U1.3 (PC15); no longer U1.1 (PB12)
- net DM: now also U2.6 (I/O1); no longer J1.A7 (D-), J1.B7 (D-)
- net DP: now also U2.4 (I/O2); no longer J1.A6 (D+), J1.B6 (D+)
- net GND: now also L_1_1.1 (K), L_1_2.1 (K), L_1_3.1 (K), L_1_4.1 (K), U2.2 (GND)
- net ROT_DOWN: now also D_1_5.1 (K); no longer SW3.B
- net ROT_UP: now also D_1_6.1 (K); no longer SW3.A
- net ROW1: now also SW3.C, D_1_4.2 (A)
- net VDD: now also U2.5 (VBUS); no longer R_1_1.1, R_1_2.1, R_1_3.1, SW3.C
- net LED3: now reaches U1.10 (PA4)
- net LED3: now also R_1_3.1
- net LED1: now reaches U1.12 (PA6)
- net LED1: now also R_1_1.1
- net COL4: now reaches U1.7 (PA1)
- net COL4: now also SW_1_4.1
- net LED4: now reaches U1.9 (PA3)
- net LED4: now also R_1_4.1
- net LED_CTRL renamed LED2
- net LED2: now also R_1_2.1
- new net: J1.A7 (D-), J1.B7 (D-), U2.1 (I/O1)
- new net: J1.A6 (D+), J1.B6 (D+), U2.3 (I/O2)
- new net: D_1_4.1 (K), SW_1_4.2
- new net: D_1_5.2 (A), SW3.A
- new net: D_1_6.2 (A), SW3.B
- new net: L_1_4.2 (A), R_1_4.2
- no-connect marks 6 -> 2
Other:
- moved on the sheet: D1, D_1_1, D_1_2, D_1_3, L_1_1, L_1_2, L_1_3, R2, R3, R5, R_1_1, R_1_2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
